Commit message: Update ranger_arm.xacro.urdf

File: urdf/ranger_arm.xacro.urdf (robot description, URDF)
Before this commit: robot ranger_arm, 47 links, 46 joints
Links:
- link arm_left_link0: geometry collision mesh filename=file://$(find libertech_ranger_arm_description)/meshes/arm/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; visual mesh filename=file://$(find libertech_ranger_arm_description)/meshes/arm/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
- link arm_left_link1: geometry collision mesh filename=file://$(find libertech_ranger_arm_description)/meshes/arm/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; visual mesh filename=file://$(find libertech_ranger_arm_description)/meshes/arm/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
- link arm_left_link2: geometry collision mesh filename=file://$(find libertech_ranger_arm_description)/meshes/arm/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; visual mesh filename=file://$(find libertech_ranger_arm_description)/meshes/arm/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
- link arm_left_link3: geometry visual mesh filename=file://$(find libertech_ranger_arm_description)/meshes/arm/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 scale=-1 1 1
- link arm_left_link4: geometry collision mesh filename=file://$(find libertech_ranger_arm_description)/meshes/arm/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; visual mesh filename=file://$(find libertech_ranger_arm_description)/meshes/arm/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
- link arm_left_link5: geometry collision mesh filename=file://$(find libertech_ranger_arm_description)/meshes/arm/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; visual mesh filename=file://$(find libertech_ranger_arm_description)/meshes/arm/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
- link arm_left_link6: geometry visual mesh filename=file://$(find libertech_ranger_arm_description)/meshes/arm/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 scale=-1 1 1
- link arm_left_link7: geometry visual mesh filename=file://$(find libertech_ranger_arm_description)/meshes/arm/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 scale=1 -1 1
- link arm_left_quick_release: geometry collision mesh filename=file://$(find libertech_ranger_arm_description)/meshes/arm/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; visual mesh filename=file://$(find libertech_ranger_arm_description)/meshes/arm/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
- link arm_right_link0: geometry collision mesh filename=file://$(find libertech_ranger_arm_description)/meshes/arm/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; visual mesh filename=file://$(find libertech_ranger_arm_description)/meshes/arm/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
- link arm_right_link1: geometry collision mesh filename=file://$(find libertech_ranger_arm_description)/meshes/arm/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; visual mesh filename=file://$(find libertech_ranger_arm_description)/meshes/arm/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
- link arm_right_link2: geometry collision mesh filename=file://$(find libertech_ranger_arm_description)/meshes/arm/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; visual mesh filename=file://$(find libertech_ranger_arm_description)/meshes/arm/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
- link arm_right_link3: geometry visual mesh filename=file://$(find libertech_ranger_arm_description)/meshes/arm/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 scale=1 1 1
- link arm_right_link4: geometry collision mesh filename=file://$(find libertech_ranger_arm_description)/meshes/arm/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; visual mesh filename=file://$(find libertech_ranger_arm_description)/meshes/arm/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
- link arm_right_link5: geometry collision mesh filename=file://$(find libertech_ranger_arm_description)/meshes/arm/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; visual mesh filename=file://$(find libertech_ranger_arm_description)/meshes/arm/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
- link arm_right_link6: geometry visual mesh filename=file://$(find libertech_ranger_arm_description)/meshes/arm/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 scale=1 1 1
- link arm_right_link7: geometry visual mesh filename=file://$(find libertech_ranger_arm_description)/meshes/arm/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 scale=1 1 1
- link arm_right_quick_release: geometry collision mesh filename=file://$(find libertech_ranger_arm_description)/meshes/arm/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; visual mesh filename=file://$(find libertech_ranger_arm_description)/meshes/arm/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
- link base_add_on: geometry collision mesh filename=file://$(find libertech_ranger_arm_description)/meshes/rang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; visual mesh filename=file://$(find libertech_ranger_arm_description)/meshes/rang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
- link base_link: geometry collision box size=0.5 0.35 0.2; visual mesh filename=file://$(find libertech_ranger_arm_description)/meshes/rang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
- link fl_steering_wheel_link: geometry collision cylinder length=0.001 radius=0.001; visual mesh filename=file://$(find libertech_ranger_arm_description)/meshes/rang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
- link fr_steering_wheel_link: geometry collision cylinder length=0.001 radius=0.001; visual mesh filename=file://$(find libertech_ranger_arm_description)/meshes/rang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
- link gripper_left_base: geometry collision mesh filename=file://$(find libertech_ranger_arm_description)/meshes/grip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; visual mesh filename=file://$(find libertech_ranger_arm_description)/meshes/grip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
- link gripper_left_finger1: geometry collision mesh filename=file://$(find libertech_ranger_arm_description)/meshes/grip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; visual mesh filename=file://$(find libertech_ranger_arm_description)/meshes/grip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
- link gripper_left_finger2: geometry collision mesh filename=file://$(find libertech_ranger_arm_description)/meshes/grip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; visual mesh filename=file://$(find libertech_ranger_arm_description)/meshes/grip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
- link gripper_right_base: geometry collision mesh filename=file://$(find libertech_ranger_arm_description)/meshes/grip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; visual mesh filename=file://$(find libertech_ranger_arm_description)/meshes/grip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
- link gripper_right_finger1: geometry collision mesh filename=file://$(find libertech_ranger_arm_description)/meshes/grip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; visual mesh filename=file://$(find libertech_ranger_arm_description)/meshes/grip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
- link gripper_right_finger2: geometry collision mesh filename=file://$(find libertech_ranger_arm_description)/meshes/grip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; visual mesh filename=file://$(find libertech_ranger_arm_description)/meshes/grip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
- link rl_steering_wheel_link: geometry collision cylinder length=0.001 radius=0.001; visual mesh filename=file://$(find libertech_ranger_arm_description)/meshes/rang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
- link rr_steering_wheel_link: geometry collision cylinder length=0.001 radius=0.001; visual mesh filename=file://$(find libertech_ranger_arm_description)/meshes/rang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

Commit message: 修改xacro文件指定方式

File: urdf/ranger_arm.xacro.urdf (robot description, URDF)
Before this commit: robot ranger_arm, 47 links, 46 joints
Links:
- link arm_left_link0: geometry collision mesh filename=https://raw.githubusercontent.com/PPML-Group/libertech_rang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; visual mesh filename=https://raw.githubusercontent.com/PPML-Group/libertech_rang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
- link arm_left_link1: geometry collision mesh filename=https://raw.githubusercontent.com/PPML-Group/libertech_rang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; visual mesh filename=https://raw.githubusercontent.com/PPML-Group/libertech_rang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
- link arm_left_link2: geometry collision mesh filename=https://raw.githubusercontent.com/PPML-Group/libertech_rang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; visual mesh filename=https://raw.githubusercontent.com/PPML-Group/libertech_rang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
- link arm_left_link3: geometry visual mesh filename=https://raw.githubusercontent.com/PPML-Group/libertech_rang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 scale=-1 1 1
- link arm_left_link4: geometry collision mesh filename=https://raw.githubusercontent.com/PPML-Group/libertech_rang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; visual mesh filename=https://raw.githubusercontent.com/PPML-Group/libertech_rang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
- link arm_left_link5: geometry collision mesh filename=https://raw.githubusercontent.com/PPML-Group/libertech_rang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; visual mesh filename=https://raw.githubusercontent.com/PPML-Group/libertech_rang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
- link arm_left_link6: geometry visual mesh filename=https://raw.githubusercontent.com/PPML-Group/libertech_rang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 scale=-1 1 1
- link arm_left_link7: geometry visual mesh filename=https://raw.githubusercontent.com/PPML-Group/libertech_rang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 scale=1 -1 1
- link arm_left_quick_release: geometry collision mesh filename=https://raw.githubusercontent.com/PPML-Group/libertech_rang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; visual mesh filename=https://raw.githubusercontent.com/PPML-Group/libertech_rang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
- link arm_right_link0: geometry collision mesh filename=https://raw.githubusercontent.com/PPML-Group/libertech_rang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; visual mesh filename=https://raw.githubusercontent.com/PPML-Group/libertech_rang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
- link arm_right_link1: geometry collision mesh filename=https://raw.githubusercontent.com/PPML-Group/libertech_rang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; visual mesh filename=https://raw.githubusercontent.com/PPML-Group/libertech_rang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
- link arm_right_link2: geometry collision mesh filename=https://raw.githubusercontent.com/PPML-Group/libertech_rang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; visual mesh filename=https://raw.githubusercontent.com/PPML-Group/libertech_rang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
- link arm_right_link3: geometry visual mesh filename=https://raw.githubusercontent.com/PPML-Group/libertech_rang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 scale=1 1 1
- link arm_right_link4: geometry collision mesh filename=https://raw.githubusercontent.com/PPML-Group/libertech_rang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; visual mesh filename=https://raw.githubusercontent.com/PPML-Group/libertech_rang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
- link arm_right_link5: geometry collision mesh filename=https://raw.githubusercontent.com/PPML-Group/libertech_rang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; visual mesh filename=https://raw.githubusercontent.com/PPML-Group/libertech_rang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
- link arm_right_link6: geometry visual mesh filename=https://raw.githubusercontent.com/PPML-Group/libertech_rang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 scale=1 1 1
- link arm_right_link7: geometry visual mesh filename=https://raw.githubusercontent.com/PPML-Group/libertech_rang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 scale=1 1 1
- link arm_right_quick_release: geometry collision mesh filename=https://raw.githubusercontent.com/PPML-Group/libertech_rang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; visual mesh filename=https://raw.githubusercontent.com/PPML-Group/libertech_rang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
- link base_add_on: geometry collision mesh filename=https://raw.githubusercontent.com/PPML-Group/libertech_rang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; visual mesh filename=https://raw.githubusercontent.com/PPML-Group/libertech_rang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
- link base_link: geometry collision box size=0.5 0.35 0.2; visual mesh filename=https://raw.githubusercontent.com/PPML-Group/libertech_rang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
- link fl_steering_wheel_link: geometry collision cylinder length=0.001 radius=0.001; visual mesh filename=https://raw.githubusercontent.com/PPML-Group/libertech_rang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
- link fr_steering_wheel_link: geometry collision cylinder length=0.001 radius=0.001; visual mesh filename=https://raw.githubusercontent.com/PPML-Group/libertech_rang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
- link gripper_left_base: geometry collision mesh filename=https://raw.githubusercontent.com/PPML-Group/libertech_rang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; visual mesh filename=https://raw.githubusercontent.com/PPML-Group/libertech_rang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
- link gripper_left_finger1: geometry collision mesh filename=https://raw.githubusercontent.com/PPML-Group/libertech_rang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; visual mesh filename=https://raw.githubusercontent.com/PPML-Group/libertech_rang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
- link gripper_left_finger2: geometry collision mesh filename=https://raw.githubusercontent.com/PPML-Group/libertech_rang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; visual mesh filename=https://raw.githubusercontent.com/PPML-Group/libertech_rang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
- link gripper_right_base: geometry collision mesh filename=https://raw.githubusercontent.com/PPML-Group/libertech_rang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; visual mesh filename=https://raw.githubusercontent.com/PPML-Group/libertech_rang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
- link gripper_right_finger1: geometry collision mesh filename=https://raw.githubusercontent.com/PPML-Group/libertech_rang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; visual mesh filename=https://raw.githubusercontent.com/PPML-Group/libertech_rang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
- link gripper_right_finger2: geometry collision mesh filename=https://raw.githubusercontent.com/PPML-Group/libertech_rang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; visual mesh filename=https://raw.githubusercontent.com/PPML-Group/libertech_rang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
- link rl_steering_wheel_link: geometry collision cylinder length=0.001 radius=0.001; visual mesh filename=https://raw.githubusercontent.com/PPML-Group/libertech_rang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
- link rr_steering_wheel_link: geometry collision cylinder length=0.001 radius=0.001; visual mesh filename=https://raw.githubusercontent.com/PPML-Group/libertech_rang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
